File: ADCS.brd (EAGLE design)
At the start: 90.2 x 95.9 mm, 434 parts, among them IC1 XC9572XL-10VQG44C, J1 SEAF-10-XX.X-XX-04-X-A, U1 Value, U10 Value, U11 Value, U12 TEXAS_INSTRUMENTS-CURRENT_MON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, U13 TEXAS_INSTRUMENTS-CURRENT_MON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, U14 Value, U15 KIOXIA_AMERICA-NAND_FLASH-TC5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, U16 KIOXIA_AMERICA-NAND_FLASH-TC5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, U17 QORVO-RF_SWITCH-QPC7512, U18 TEXAS_INSTRUMENTS-CURRENT_MON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, U19 TEXAS_INSTRUMENTS-BUCK_CONVER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, U2 Value, U20 Value, U21 Value, U22 Value, U23 TEXAS_INSTRUMENTS-AND_GATE-SN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, U24 KIOXIA_AMERICA-NAND_FLASH-TC5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, U3 Value, U34 TMP100, U4 Value, U5 TEXAS_INSTRUMENTS-AND_GATE-SN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, U6 ISSI-DRAM-IS42S16320F-7TL, U7 TMP100, U8 BMX160, U9 BMX160, X1 ECS_INC-OSCILLATOR-ECS-400-10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, X2 BU-SMA-V, X3 2510-, X4 2510-, X5 2510-, X6 5566-4, X7 ECS_INC-OSCILLATOR-ECS-400-10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, X8 2510-, Y1 20MHz, Y2 20MHz, Y3 20MHz

Commit message: PCB routing progress
Parts:
- C257, C258, C259, C260, C261, C262, C263, L14, L15, L16, L17, L18, L19, L20: device standardparts:0603 -> standardparts:0402
- moved JP8 212.3 mm to (87.0, 22.9), turned to 90 degrees
- moved JP7 208.4 mm to (87.0, 16.5), turned to 90 degrees
- moved JP6 204.9 mm to (87.0, 10.2), turned to 90 degrees
- moved JP5 201.7 mm to (87.0, 3.81), turned to 90 degrees
- moved C261 199.1 mm to (65.5, 77.0)
- moved C259 197.4 mm to (70.6, 73.2), turned to 180 degrees
- moved C260 197.2 mm to (66.8, 74.2)
- moved C258 194.1 mm to (70.6, 71.4)
- moved C59 189.5 mm to (55.9, 93.0), flipped to the bottom
- moved C213 187.9 mm to (55.9, 82.3), turned to 180 degrees
- moved C257 187.9 mm to (67.8, 70.6)
- moved C56 186.0 mm to (60.2, 94.5), turned to 180 degrees
- moved C58 184.6 mm to (52.6, 89.4), flipped to the bottom
- moved C54 184.0 mm to (62.2, 89.9), flipped to the bottom
- moved C57 181.5 mm to (52.3, 90.9), flipped to the bottom
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Routing:
- net VSS: track 76.1 -> 142.2 mm, vias 91 -> 131
- net VCC_3V3_IO: track 44.0 -> 98.5 mm, vias 26 -> 48
- net TRX2_SW: track 0.00 -> 11.0 mm
- net LNA2_P: track 0.00 -> 8.77 mm
- net LNA2_N: track 0.00 -> 8.73 mm
- net PA: track 8.17 -> 16.2 mm
- net N$51: track 0.00 -> 7.11 mm
- net N$52: track 0.00 -> 5.54 mm
- net N$56: track 0.00 -> 4.96 mm
- net !CC1200_2_RESET: track 0.00 -> 4.91 mm, vias 0 -> 1
- net N$72: track 0.00 -> 4.52 mm
- net N$70: track 0.00 -> 4.42 mm
- net N$71: track 0.00 -> 4.02 mm
- net ANT2_PREMUX_50Z: track 0.00 -> 3.79 mm
- net N$55: track 0.00 -> 3.69 mm
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
Commit message: PCB progress and schematic checking
Connections:
- net !COMMS1_UNRESPONSIVE renamed !COMMS1_UNRESPONSIVE_FROM_SMC
- net !COMMS2_UNRESPONSIVE renamed !COMMS2_UNRESPONSIVE_FROM_SMC
- net !SMC_UNRESPONSIVE1 renamed !SMC_UNRESPONSIVE_FROM_COMMS1
- net !SMC_UNRESPONSIVE2 renamed !SMC_UNRESPONSIVE_FROM_COMMS2
- net SMC_ERR_OUT_CPLD renamed SMC_ERR_CPLD_IN
