File: ADCS.sch (EAGLE design)
At the start: 434 parts, among them IC1 XC9572XL-10VQG44C, J1 SEAF-10-XX.X-XX-04-X-A, U1 Value, U10 Value, U11 Value, U12 TEXAS_INSTRUMENTS-CURRENT_MON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, U13 TEXAS_INSTRUMENTS-CURRENT_MON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, U14 Value, U15 KIOXIA_AMERICA-NAND_FLASH-TC5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, U16 KIOXIA_AMERICA-NAND_FLASH-TC5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, U17 QORVO-RF_SWITCH-QPC7512, U18 TEXAS_INSTRUMENTS-CURRENT_MON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, U19 TEXAS_INSTRUMENTS-BUCK_CONVER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, U2 Value, U20 Value, U21 Value, U22 Value, U23 TEXAS_INSTRUMENTS-AND_GATE-SN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, U24 KIOXIA_AMERICA-NAND_FLASH-TC5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, U3 Value, U34 TMP100, U4 Value, U5 TEXAS_INSTRUMENTS-AND_GATE-SN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, U6 ISSI-DRAM-IS42S16320F-7TL, U7 TMP100, U8 BMX160, U9 BMX160, X1 ECS_INC-OSCILLATOR-ECS-400-10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, X2 BU-SMA-V, X3 2510-, X4 2510-, X5 2510-, X6 5566-4, X7 ECS_INC-OSCILLATOR-ECS-400-10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, X8 2510-, Y1 20MHz, Y2 20MHz, Y3 20MHz

Commit message: PCB routing progress
Parts:
- C257, C258, C259, C260, C261, C262, C263: device standardparts:CAPACITOR.0603 -> standardparts:CAPACITOR.0402
- L14, L15, L16, L17, L18, L19, L20: device standardparts:RF-INDUCTOR.0603 -> standardparts:RF-INDUCTOR.0402
Changed lines of the file:
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@@
 <part name="C256" library="standardparts" deviceset="CAPACITOR" device=".0603" value="1uF"/>
 <part name="S259" library="Module_Supplies" deviceset="VSS" device=""/>
-<part name="C257" library="standardparts" deviceset="CAPACITOR" device=".0603" value="15pF"/>
-<part name="L14" library="standardparts" deviceset="RF-INDUCTOR" device=".0603" value="7.5nH"/>
-<part name="C258" library="standardparts" deviceset="CAPACITOR" device=".0603" value="1pF"/>
-<part name="L15" library="standardparts" deviceset="RF-INDUCTOR" device=".0603" value="18nH"/>
-<part name="C259" library="standardparts" deviceset="CAPACITOR" device=".0603" value="2.2pF"/>
-<part name="L16" library="standardparts" deviceset="RF-INDUCTOR" device=".0603" value="12nH"/>
-<part name="L17" library="standardparts" deviceset="RF-INDUCTOR" device=".0603" value="12nH"/>
-<part name="C260" library="standardparts" deviceset="CAPACITOR" device=".0603" value="3.3pF"/>
-<part name="L18" library="standardparts" deviceset="RF-INDUCTOR" device=".0603" value="15nH"/>
-<part name="C261" library="standardparts" deviceset="CAPACITOR" device=".0603" value="3.3pF"/>
-<part name="L19" library="standardparts" deviceset="RF-INDUCTOR" device=".0603" value="12nH"/>
+<part name="C257" library="standardparts" deviceset="CAPACITOR" device=".0402" value="15pF"/>
+<part name="L14" library="standardparts" deviceset="RF-INDUCTOR" device=".0402" value="7.5nH"/>
+<part name="C258" library="standardparts" deviceset="CAPACITOR" device=".0402" value="1pF"/>
+<part name="L15" library="standardparts" deviceset="RF-INDUCTOR" device=".0402" value="18nH"/>
+<part name="C259" library="standardparts" deviceset="CAPACITOR" device=".0402" value="2.2pF"/>
+<part name="L16" library="standardparts" deviceset="RF-INDUCTOR" device=".0402" value="12nH"/>
+<part name="L17" library="standardparts" deviceset="RF-INDUCTOR" device=".0402" value="12nH"/>
+<part name="C260" library="standardparts" deviceset="CAPACITOR" device=".0402" value="3.3pF"/>
+<part name="L18" library="standardparts" deviceset="RF-INDUCTOR" device=".0402" value="15nH"/>
+<part name="C261" library="standardparts" deviceset="CAPACITOR" device=".0402" value="3.3pF"/>
+<part name="L19" library="standardparts" deviceset="RF-INDUCTOR" device=".0402" value="12nH"/>
 <part name="S260" library="Module_Supplies" deviceset="VSS" device=""/>
-<part name="C262" library="standardparts" deviceset="CAPACITOR" device=".0603" value="3pF"/>
+<part name="C262" library="standardparts" deviceset="CAPACITOR" device=".0402" value="3pF"/>
 <part name="S261" library="Module_Supplies" deviceset="VSS" device=""/>
-<part name="L20" library="standardparts" deviceset="RF-INDUCTOR" device=".0603" value="12nH"/>
-<part name="C263" library="standardparts" deviceset="CAPACITOR" device=".0603" value="DNI"/>
+<part name="L20" library="standardparts" deviceset="RF-INDUCTOR" device=".0402" value="12nH"/>
+<part name="C263" library="standardparts" deviceset="CAPACITOR" device=".0402" value="DNI"/>
 <part name="U24" library="Module_ICs" deviceset="KIOXIA_AMERICA-NAND_FLASH-TC58CVG0S3HRAIG" device="" package3d_urn="urn:adsk.eagle:package:14910091/1"/>
 <part name="S262" library="Module_Supplies" deviceset="VSS" device=""/>

Commit message: PCB progress and schematic checking
Connections:
- net !COMMS1_UNRESPONSIVE renamed !COMMS1_UNRESPONSIVE_FROM_SMC
- net !COMMS2_UNRESPONSIVE renamed !COMMS2_UNRESPONSIVE_FROM_SMC
- net !SMC_UNRESPONSIVE1 renamed !SMC_UNRESPONSIVE_FROM_COMMS1
- net !SMC_UNRESPONSIVE2 renamed !SMC_UNRESPONSIVE_FROM_COMMS2
- net SMC_ERR_OUT_CPLD renamed SMC_ERR_CPLD_IN
