File: Design Files/OBC.sch (EAGLE design)
At the start: 118 parts, among them U1 STMICROELECTRONICS-MICROCONTR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, U10 Value, U11 Value, U12 TEXAS_INSTRUMENTS-CURRENT_MON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, U13 TEXAS_INSTRUMENTS-CURRENT_MON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, U17 QORVO-RF_SWITCH-QPC7512, U18 TEXAS_INSTRUMENTS-CURRENT_MON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, U19 TEXAS_INSTRUMENTS-BUCK_CONVER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, U34 TMP100, U7 TMP100, U8 BMX160, U9 BMX160, X2 BU-SMA-V, X6 5566-4

Commit message: Schematic progress
Parts:
- added C16, C17, C18, C19, C20, C21, C39, C42: 0.1uF, standardparts:CAPACITOR.0603
- added C22, C23, C24: 1uF, standardparts:CAPACITOR.0603
- added C25, C26: 4.7uF, standardparts:CAPACITOR.0603
- added C27, C28, C34, C35, C36: DNI, standardparts:CAPACITOR.0402
- added C29, C30, C33: 2.7pF, standardparts:CAPACITOR.0402
- added C31: 6.2pF, standardparts:CAPACITOR.0402
- added C32: 3.6pF, standardparts:CAPACITOR.0402
- added C37, C38, C40, C41: 20pF, standardparts:CAPACITOR.0603
- added JTAG1: (no value), microbuilder:JTAG-CORTEXM3MOLEX
- added L1, L2, L3, L4: 18nH, standardparts:RF-INDUCTOR.0402
- added L5, L6: 12nH, standardparts:RF-INDUCTOR.0402
- added L7: 0R, standardparts:RF-INDUCTOR.0402
- added R1, R4, R5, R6: 10k, standardparts:RESISTOR.0603
- added R2: DNI, standardparts:RESISTOR.0603
- added R3: 47k, standardparts:RESISTOR.0603
- added R7: 0R, standardparts:RESISTOR.0603
- added U2: ON_SEMICONDUCTOR-RF_TRANSCEIVER-AX5043, Module_ICs:ON_SEMICONDUCTOR-RF_TRANSCEIVER-AX5043
- added U3: Value, Module_Gates:TEXAS_INSTRUMENTS-AND_GATE-SN74LVC1G08DBVR
- added U4: STMICROELECTRONICS-MICROCONTROLLER-STM32F412ZGT6TR, Module_ICs:STMICROELECTRONICS-MICROCONTROLLER-STM32F412ZGT6TR
- added X1, X3: 16MHz, Module_ICs:ECS_INC-OSCILLATOR-ECS-160-20-23A-TR
- added X4: (no value), Module_ICs:ECS_INC-OSCILLATOR-ECS-.327-12.5-1210B-N-TR
- U1: value STMICROELECTRONICS-MICROCONTROLLER-STM32L010R8T6 -> STMICROELECTRONICS-MICROCONTROLLER-STM32L431RCT6; device Module_ICs:STMICROELECTRONICS-MICROCONTROLLER-STM32L010R8T6 -> Module_ICs:STMICROELECTRONICS-MICROCONTROLLER-STM32L431RCT6
Connections:
- new net !COMMS1_JTAG_RESET: JTAG1.10, R6.2, U3.B
- new net !COMMS1_NRST_IN: R4.2, U1A.NRST, U3.Y
- new net !COMMS1_RESET: R5.2, U3.A
- new net !COMMS1_RF_SPI_CS: R1.1, U1A.PA4, U2.SEL
- new net COMMS1_BOOT0: R2.2, R3.1, U1A.PH3/BOOT0
- new net COMMS1_JTAG_TCK: JTAG1.4
- new net COMMS1_JTAG_TDI: JTAG1.8
- new net COMMS1_JTAG_TDO: JTAG1.6
- new net COMMS1_JTAG_TMS: JTAG1.2
- new net COMMS1_RF_INT: U2.IRQ
- new net COMMS1_RF_SPI_MISO: U1A.PA6, U2.MISO
- new net COMMS1_RF_SPI_MOSI: U1A.PA7, U2.MOSI
- new net COMMS1_RF_SPI_SCK: U1A.PA5, U2.CLK
- new net HFOSC_XI: C40.1, U1A.PH0-OSC_IN, X3.XI
- new net HFOSC_XO: C41.1, U1A.PH1-OSC_OUT, X3.XO
- new net LFOSC_XI: U1A.PC14-OSC32_IN, X4.XO
- new net LFOSC_XO: U1A.PC15-OSC32_OUT, X4.XI
- new net N$1: U2.L1, U2.L2
- new net N$11: C38.2, U2.CLK16N, X1.XO
- new net N$17: C42.1, R7.2, U1B.VBAT
- new net N$2: C32.1, C33.2, L4.1, L5.2
- new net N$3: C29.1, L3.2
- new net N$4: C27.1, C29.2, L1.2, U2.ANTP
- new net N$5: C28.1, C30.2, L2.2, U2.ANTN
- new net N$6: C30.1, L4.2
- new net N$7: C31.1, L3.1, L6.2
- new net N$8: C37.2, U2.CLK16P, X1.XI
- new net N$9: C33.1, C34.1, C36.2, L6.1, L7.2
- net ANT1_PREMUX_50Z: now also C35.1, C36.1, L7.1
- net VCC_3V3_IO: now also C16.1, C17.1, C18.1, C19.1, C20.1, C21.1, C22.1, C23.1, C24.1, C25.1, C26.1, C39.1, JTAG1.1, R2.1, R4.1, R5.1, R6.1, R7.1, U1B.VDDA/VREF+, U2.VDD_ANA@1, U2.VDD_ANA@2, U2.VDD_IO@1, U3.V+; no longer U1B.VDDA, U1B.VDDIO2
- net VSS: now also C16.2, C17.2, C18.2, C19.2, C20.2, C21.2, C22.2, C23.2, C24.2, C25.2, C26.2, C27.2, C28.2, C31.2, C32.2, C34.2, C35.2, C37.1, C38.1, C39.2, C40.2, C41.2, C42.2, JTAG1.3, JTAG1.5, JTAG1.9, L1.1, L2.1, L5.1, R1.2, R3.2, U1B.VSSA/VREF-, U2.GND@1, U2.GND@2, U2.GPADC1, U2.GPADC2, U3.V-, X4.VSS; no longer U1B.VSSA
Other:
- note added: "MCU Power Block"
- note added: "Note: 0R indicates placement of a 0 ohm bridge resistor in place of the inductor"
- note added: "Note: 50 ohm impedance for all RF traces"
- note added: "Note: 868/915 MHz operation"
- note added: "Note: for DNI values, reference the AX5043 datasheet"
- note added: "Single-ended RF transceiver"
- moved on the sheet: U1B
